Commit message: initial test configuration setup

File: urdf/arm/openarm_arm.xacro (robot description, xacro)
@@ -4,9 +4,12 @@
   <xacro:macro name="openarm_arm" params="arm_type arm_prefix:='' no_prefix:=false description_pkg:='openarm_description' connected_to:='base' xyz:='0 0 0' rpy:='0 0 0' joint_limits inertials kinematics kinematics_link kinematics_offset:=none " >
     <xacro:property name="prefix" value="${'' if no_prefix else 'openarm' + '_' + arm_prefix}" />
-    <xacro:if value="${arm_prefix == 'right_'}">
+    <!-- reflect=+1 for right arm (explicit "right_" prefix) and for single arm
+         (empty prefix), which is always right-arm hardware.
+         reflect=-1 only for the explicitly mirrored left arm ("left_" prefix). -->
+    <xacro:if value="${arm_prefix == 'left_'}">
+      <xacro:property name="reflect" value="-1" />
+    </xacro:if>
+    <xacro:unless value="${arm_prefix == 'left_'}">
       <xacro:property name="reflect" value="1" />
-    </xacro:if>
-    <xacro:unless value="${arm_prefix == 'right_'}">
-      <xacro:property name="reflect" value="-1" />
     </xacro:unless>
     <xacro:unless value="${connected_to == ''}">
@@ -79,5 +82,9 @@
       <parent link="${prefix}link6"/>
       <child link="${prefix}link7"/>
-      <axis xyz="0 ${reflect} 0"/>
+      <!-- J7 hardware positive direction is +Y for single arm (empty prefix) and
+           right arm (right_ prefix).  Left arm (left_ prefix) uses -Y via reflect=-1.
+           This matches the original axis assignment for all three configurations. -->
+      <xacro:property name="j7_sign" value="${reflect}"/>
+      <axis xyz="0 ${j7_sign} 0"/>
       <xacro:openarm-limits name="joint7" config="${joint_limits}" />
     </joint>

File: urdf/robot/openarm_robot.xacro (robot description, xacro)
@@ -37,5 +37,8 @@
             left_arm_prefix:='left_'
             right_arm_prefix:='right_'
-            can_fd:='true'
+            can_fd:='false'
+            with_body:='false'
+            arm_base_xyz:='0.0 -0.031 0.698'
+            arm_base_rpy:='1.5708 0 0'
             "
             >
@@ -136,4 +139,33 @@
     </xacro:if>
     <xacro:if value="${not bimanual}">
+        <!-- Single arm with body/rod mount (world → openarm_body_link0 → arm) -->
+        <xacro:if value="${with_body}">
+          <xacro:openarm_body
+            body_type="${body_type}"
+            body_prefix="${body_prefix_modified}"
+            no_prefix="${no_prefix}"
+            description_pkg="openarm_description"
+            connected_to="${body_connected_to}"
+            xyz="${xyz}"
+            rpy="${rpy}"
+            inertials="${body_inertials}"
+            kinematics="${body_kinematics}"
+            kinematics_link="${body_kinematics_link}" />
+          <xacro:openarm_arm
+            arm_type="${arm_type}"
+            arm_prefix="${arm_prefix_modified}"
+            no_prefix="${no_prefix}"
+            description_pkg="openarm_description"
+            connected_to="openarm_body_link0"
+            xyz="${arm_base_xyz}"
+            rpy="${arm_base_rpy}"
+            joint_limits="${joint_limits}"
+            kinematics="${kinematics}"
+            kinematics_link="${kinematics_link}"
+            inertials="${inertials}"
+            kinematics_offset="${kinematics_offset}" />
+        </xacro:if>
+        <!-- Single arm standalone (floating, no body) -->
+        <xacro:if value="${not with_body}">
         <xacro:openarm_arm
         arm_type="${arm_type}"
@@ -148,4 +180,5 @@
         connected_to=""
         />
+        </xacro:if>
         <xacro:if value="${ros2_control}">
         <xacro:openarm_arm_ros2_control

Commit message: correct canport for the arms and urdf correction

File: urdf/arm/openarm_arm.xacro (robot description, xacro)
@@ -82,9 +82,5 @@
       <parent link="${prefix}link6"/>
       <child link="${prefix}link7"/>
-      <!-- J7 hardware positive direction is +Y for single arm (empty prefix) and
-           right arm (right_ prefix).  Left arm (left_ prefix) uses -Y via reflect=-1.
-           This matches the original axis assignment for all three configurations. -->
-      <xacro:property name="j7_sign" value="${reflect}"/>
-      <axis xyz="0 ${j7_sign} 0"/>
+      <axis xyz="0 ${reflect} 0"/>
       <xacro:openarm-limits name="joint7" config="${joint_limits}" />
     </joint>

File: urdf/robot/v10.urdf.xacro (robot description, xacro)
@@ -15,6 +15,6 @@
   <xacro:arg name="ros2_control" default="false" />
   <xacro:arg name="can_interface" default="slcan0" />
-  <xacro:arg name="left_can_interface" default="can1" />
-  <xacro:arg name="right_can_interface" default="slcan0" />
+  <xacro:arg name="left_can_interface" default="can0" />
+  <xacro:arg name="right_can_interface" default="can1" />
   <xacro:arg name="left_arm_prefix" default="left_" />
   <xacro:arg name="right_arm_prefix" default="right_" />

File: urdf/ros2_control/openarm.bimanual.ros2_control.xacro (robot description, xacro)
@@ -4,6 +4,6 @@
          params="arm_type
              control_gains
-             left_can_interface:=^|can1
-             right_can_interface:=^|can0
+             left_can_interface:=^|can0
+             right_can_interface:=^|can1
              use_fake_hardware:=^|false
              fake_sensor_commands:=^|false
